File: 42_project_00/42_project_00.kicad_pcb (KiCad board)
At the start: 2 copper layers, 21 x 31.1 mm, 17 parts, among them J3 FTDI, SW1 SW_Push, U1 ATmega328p-A, Y1 16Mhz

Commit message: bonus done, diferential pairs ?
Parts:
- added G***: LOGO, Custom_logos:eiffel, F.Cu at (134.3, 39.2)
- added G***: LOGO, Custom_logos:ardu42, B.Cu at (138.7, 37.5)
- C1, C2, C4, C5, C6, C7: footprint MyFootLib:0603_CA -> MyFootLib:0603_CA_C
- D1, D2: footprint MyFootLib:0603_CA -> MyFootLib:0603_CA_D
- R1, R2, R3: footprint MyFootLib:0603_CA -> MyFootLib:0603_CA_R
- moved C6 2.60 mm to (135.3, 43.1)
- moved C7 2.60 mm to (133.3, 43.1)
- moved R3 1.30 mm to (134.3, 45.8)
- moved R2 0.30 mm to (134.3, 47.6)
Routing:
- net GND: track 82.3 -> 15.2 mm, vias 4 -> 5
- net RXI: track 35.9 -> 33.1 mm
- net DTR: track 45.0 -> 43.3 mm
- net RAW: track 61.0 -> 59.9 mm, vias 3 -> 2
- net D4: track 25.1 -> 24.1 mm
- net D3: track 23.8 -> 22.9 mm
- net A2: track 8.31 -> 9.01 mm
- net MISO: track 14.4 -> 13.7 mm
- net SCK: track 55.8 -> 55.2 mm
- added copper zone on B.Cu, net GND
- added copper zone on F.Cu, net GND
Other:
- board size 21 x 31.1 mm -> 21.3 x 31.6 mm
