File: 42_project_00/42_project_00.kicad_sch (KiCad schematic)
At the start: 29 parts, among them J3 FTDI, SW1 SW_Push, U1 ATmega328p-A, Y1 16Mhz

Commit message: mandatory done, check RAW
Parts:
- removed GND1, GND2, GND3, GND4, GND5, GND6, GND7, GND8: ~, symbol New_Library:GND
- removed VCC1, VCC2, VCC3, VCC4: ~, symbol New_Library:VCC
- C1, C2, C4, C5, C6, C7, D1, D2, R1, R2, R3: footprint (none) -> MyFootLib:0603_CA
- J1, J2: footprint (none) -> MyFootLib:SidePorts
- J3: footprint (none) -> MyFootLib:FTDI
- SW1: footprint (none) -> MyFootLib:Omron_B3U-1000P
- U1: footprint (none) -> MyFootLib:ATmega328p-AU
- Y1: footprint (none) -> MyFootLib:Crystal
Connections:
- net RAW is gone; now on net VCC: C6.1, C7.1, D2.1, J2.1
- net GND: now also C1.2, C2.2, C4.1, C6.2, C7.2, D1.2, R2.1, U1.3 (GND), Y1.2, Y1.4
- net VCC: now also C5.1, R3.2, U1.18 (AVCC), U1.4 (VCC)

Commit message: bonus done, diferential pairs ?
Parts:
- C1, C2, C4, C5, C6, C7: footprint MyFootLib:0603_CA -> MyFootLib:0603_CA_C
- D1, D2: footprint MyFootLib:0603_CA -> MyFootLib:0603_CA_D
- R1, R2, R3: footprint MyFootLib:0603_CA -> MyFootLib:0603_CA_R
Changed lines of the file:
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@@
 			)
 		)
-		(property "Footprint" "MyFootLib:0603_CA"
+		(property "Footprint" "MyFootLib:0603_CA_R"
 			(at 69.85 26.67 0)
 			(effects
@@
 			)
 		)
-		(property "Footprint" "MyFootLib:0603_CA"
+		(property "Footprint" "MyFootLib:0603_CA_D"
 			(at 69.85 33.02 0)
 			(effects
@@
 			)
 		)
-		(property "Footprint" "MyFootLib:0603_CA"
+		(property "Footprint" "MyFootLib:0603_CA_R"
 			(at 44.45 36.83 0)
 			(effects
@@
 			)
 		)
-		(property "Footprint" "MyFootLib:0603_CA"
+		(property "Footprint" "MyFootLib:0603_CA_C"
 			(at 39.37 77.47 0)
 			(effects
@@
 			)
 		)
-		(property "Footprint" "MyFootLib:0603_CA"
+		(property "Footprint" "MyFootLib:0603_CA_D"
 			(at 44.45 30.48 0)
 			(effects
@@
 			)
 		)
-		(property "Footprint" "MyFootLib:0603_CA"
+		(property "Footprint" "MyFootLib:0603_CA_C"
 			(at 27.94 34.29 0)
 			(effects
@@
 			)
 		)
-		(property "Footprint" "MyFootLib:0603_CA"
+		(property "Footprint" "MyFootLib:0603_CA_C"
 			(at 78.74 85.09 0)
 			(effects
@@
 			)
 		)
-		(property "Footprint" "MyFootLib:0603_CA"
+		(property "Footprint" "MyFootLib:0603_CA_C"
 			(at 78.74 95.25 0)
 			(effects
@@
 			)
 		)
-		(property "Footprint" "MyFootLib:0603_CA"
+		(property "Footprint" "MyFootLib:0603_CA_C"
 			(at 35.56 34.29 0)
 			(effects
@@
 			)
 		)
-		(property "Footprint" "MyFootLib:0603_CA"
+		(property "Footprint" "MyFootLib:0603_CA_C"
 			(at 96.52 35.56 0)
 			(effects
@@
 			)
 		)
-		(property "Footprint" "MyFootLib:0603_CA"
+		(property "Footprint" "MyFootLib:0603_CA_R"
 			(at 113.03 30.48 0)
 			(effects

Commit message: new names, kicad_sch warning?
Parts:
- C1, C2, C4, C5, C6, C7: symbol New_Library:Capacitor -> MySymbolLib:Capacitor
- D1, D2: symbol New_Library:LED -> MySymbolLib:LED
- J1, J2: symbol New_Library:J_port -> MySymbolLib:J_port
- J3: symbol New_Library:FTDI -> MySymbolLib:FTDI
- R1, R2, R3: symbol New_Library:Resistor -> MySymbolLib:Resistor
- SW1: symbol New_Library:PushButton -> MySymbolLib:PushButton
- U1: symbol New_Library:ATmega328p -> MySymbolLib:ATmega328p
- Y1: symbol New_Library:4PIN_Crystal -> MySymbolLib:4PIN_Crystal
Changed lines of the file:
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@@
 	)
 	(symbol
-		(lib_id "New_Library:Resistor")
+		(lib_id "MySymbolLib:Resistor")
 		(at 69.85 26.67 90)
 		(unit 1)
@@
 	(symbol
 		(lib_name "GND_1")
-		(lib_id "New_Library:GND")
+		(lib_id "MySymbolLib:GND")
 		(at 69.85 39.37 0)
 		(unit 1)
@@
 	)
 	(symbol
-		(lib_id "New_Library:LED")
+		(lib_id "MySymbolLib:LED")
 		(at 69.85 33.02 270)
 		(unit 1)
@@
 	(symbol
 		(lib_name "VCC_2")
-		(lib_id "New_Library:VCC")
+		(lib_id "MySymbolLib:VCC")
 		(at 113.03 24.13 0)
 		(unit 1)
@@
 	)
 	(symbol
-		(lib_id "New_Library:Resistor")
+		(lib_id "MySymbolLib:Resistor")
 		(at 44.45 36.83 90)
 		(unit 1)
@@
 	)
 	(symbol
-		(lib_id "New_Library:J_port")
+		(lib_id "MySymbolLib:J_port")
 		(at 99.06 87.63 0)
 		(unit 1)
@@
 	(symbol
 		(lib_name "GND_1")
-		(lib_id "New_Library:GND")
+		(lib_id "MySymbolLib:GND")
 		(at 35.56 40.64 0)
 		(unit 1)
@@
 	(symbol
 		(lib_name "VCC_3")
-		(lib_id "New_Library:VCC")
+		(lib_id "MySymbolLib:VCC")
 		(at 35.56 73.66 0)
 		(unit 1)
@@
 	)
 	(symbol
-		(lib_id "New_Library:Capacitor")
+		(lib_id "MySymbolLib:Capacitor")
 		(at 39.37 77.47 0)
 		(unit 1)
@@
 	)
 	(symbol
-		(lib_id "New_Library:LED")
+		(lib_id "MySymbolLib:LED")
 		(at 44.45 30.48 270)
 		(unit 1)
@@
 	)
 	(symbol
-		(lib_id "New_Library:4PIN_Crystal")
+		(lib_id "MySymbolLib:4PIN_Crystal")
 		(at 73.66 90.17 0)
 		(unit 1)
@@
 	)
 	(symbol
-		(lib_id "New_Library:Capacitor")
+		(lib_id "MySymbolLib:Capacitor")
 		(at 27.94 34.29 270)
 		(unit 1)
@@
 	)
 	(symbol
-		(lib_id "New_Library:Capacitor")
+		(lib_id "MySymbolLib:Capacitor")
 		(at 78.74 85.09 0)
 		(unit 1)
@@
 	)
 	(symbol
-		(lib_id "New_Library:VCC")
+		(lib_id "MySymbolLib:VCC")
 		(at 53.34 69.85 0)
 		(unit 1)
@@
 	)
 	(symbol
-		(lib_id "New_Library:Capacitor")
+		(lib_id "MySymbolLib:Capacitor")
 		(at 78.74 95.25 0)
 		(unit 1)
@@
 	)
 	(symbol
-		(lib_id "New_Library:VCC")
+		(lib_id "MySymbolLib:VCC")
 		(at 142.24 35.56 180)
 		(unit 1)
@@
 	)
 	(symbol
-		(lib_id "New_Library:#PWR")
+		(lib_id "MySymbolLib:#PWR")
 		(at 134.62 31.75 90)
 		(unit 1)
@@
 	(symbol
 		(lib_name "VCC_1")
-		(lib_id "New_Library:VCC")
+		(lib_id "MySymbolLib:VCC")
 		(at 44.45 22.86 0)
 		(unit 1)
@@
 	(symbol
 		(lib_name "GND_2")
-		(lib_id "New_Library:GND")
+		(lib_id "MySymbolLib:GND")
 		(at 134.62 35.56 0)
 		(unit 1)
@@
 	)
 	(symbol
-		(lib_id "New_Library:J_port")
+		(lib_id "MySymbolLib:J_port")
 		(at 118.11 96.52 180)
 		(unit 1)
@@
 	)
 	(symbol
-		(lib_id "New_Library:Capacitor")
+		(lib_id "MySymbolLib:Capacitor")
 		(at 35.56 34.29 270)
 		(unit 1)
@@
 	(symbol
 		(lib_name "GND_2")
-		(lib_id "New_Library:GND")
+		(lib_id "MySymbolLib:GND")
 		(at 67.31 91.44 0)
 		(unit 1)
@@
 	(symbol
 		(lib_name "GND_2")
-		(lib_id "New_Library:GND")
+		(lib_id "MySymbolLib:GND")
 		(at 83.82 91.44 0)
 		(unit 1)
@@
 	(symbol
 		(lib_name "GND_1")
-		(lib_id "New_Library:GND")
+		(lib_id "MySymbolLib:GND")
 		(at 44.45 43.18 0)
 		(unit 1)
@@
 	)
 	(symbol
-		(lib_id "New_Library:#PWR")
+		(lib_id "MySymbolLib:#PWR")
 		(at 142.24 31.75 90)
 		(unit 1)
@@
 	)
 	(symbol
-		(lib_id "New_Library:PushButton")
+		(lib_id "MySymbolLib:PushButton")
 		(at 105.41 35.56 0)
 		(unit 1)
@@
 	)
 	(symbol
-		(lib_id "New_Library:ATmega328p")
+		(lib_id "MySymbolLib:ATmega328p")
 		(at 55.88 93.98 0)
 		(unit 1)
@@
 	)
 	(symbol
-		(lib_id "New_Library:FTDI")
+		(lib_id "MySymbolLib:FTDI")
 		(at 127 88.9 0)
 		(unit 1)
@@
 	)
 	(symbol
-		(lib_id "New_Library:Capacitor")
+		(lib_id "MySymbolLib:Capacitor")
 		(at 96.52 35.56 0)
 		(unit 1)
@@
 	)
 	(symbol
-		(lib_id "New_Library:Resistor")
+		(lib_id "MySymbolLib:Resistor")
 		(at 113.03 30.48 90)
 		(unit 1)
@@
 	(symbol
 		(lib_name "GND_1")
-		(lib_id "New_Library:GND")
+		(lib_id "MySymbolLib:GND")
 		(at 91.44 39.37 0)
 		(unit 1)
@@
 	)
 	(symbol
-		(lib_id "New_Library:GND")
+		(lib_id "MySymbolLib:GND")
 		(at 27.94 40.64 0)
 		(unit 1)
@@
 	(symbol
 		(lib_name "GND_2")
-		(lib_id "New_Library:GND")
+		(lib_id "MySymbolLib:GND")
 		(at 52.07 114.3 0)
 		(unit 1)
